Commit message: release astribot_descriptions_github @ v0.0.0-dev

File: astribot_t1/model/urdf/astribot_head.urdf (robot description, URDF)
Before this commit: robot astribot_head, 3 links, 2 joints
Joints:
- joint astribot_head_joint_1: limit lower=-1.611 upper=1.605 effort=15.0 velocity=2.0 -> lower=-1.608 upper=1.608 effort=15.0 velocity=2.0
- joint astribot_head_joint_2: limit lower=-0.583 upper=0.534 effort=15.0 velocity=2.0 -> lower=-0.558 upper=0.558 effort=15.0 velocity=2.0

File: astribot_t1/model/urdf/astribot_whole_body.urdf (robot description, URDF)
Before this commit: robot astribot_t1, 47 links, 46 joints
Joints:
- joint astribot_head_joint_1: limit lower=-1.611 upper=1.605 effort=15.0 velocity=2.0 -> lower=-1.608 upper=1.608 effort=15.0 velocity=2.0
- joint astribot_head_joint_2: limit lower=-0.583 upper=0.534 effort=15.0 velocity=2.0 -> lower=-0.558 upper=0.558 effort=15.0 velocity=2.0
