Commit message: release astribot_descriptions_github @ v0.0.0-dev

File: astribot_t1/model/urdf/astribot_arm_left.urdf (robot description, URDF)
Before this commit: robot astribot_arm_left, 9 links, 8 joints
Joints:
- joint astribot_arm_left_joint_5: limit lower=-2.103 upper=2.098 effort=20.0 velocity=10.0 -> lower=-2.101 upper=2.101 effort=20.0 velocity=10.0
- joint astribot_arm_left_joint_6: limit lower=-0.755 upper=0.744 effort=8.0 velocity=5.0 -> lower=-0.75 upper=0.75 effort=8.0 velocity=5.0
- joint astribot_arm_left_joint_7: limit lower=-1.449 upper=1.485 effort=8.0 velocity=5.0 -> lower=-1.467 upper=1.467 effort=8.0 velocity=5.0

File: astribot_t1/model/urdf/astribot_arm_right.urdf (robot description, URDF)
Before this commit: robot astribot_arm_right, 9 links, 8 joints
Joints:
- joint astribot_arm_right_joint_1: limit lower=-1.606 upper=3.158 effort=80.0 velocity=3.0 -> lower=-1.579 upper=3.172 effort=80.0 velocity=3.0
- joint astribot_arm_right_joint_2: limit lower=-1.539 upper=0.192 effort=80.0 velocity=3.0 -> lower=-1.538 upper=0.201 effort=80.0 velocity=3.0
- joint astribot_arm_right_joint_3: limit lower=-0.741 upper=2.331 effort=40.0 velocity=3.0 -> lower=-0.745 upper=2.321 effort=40.0 velocity=3.0
- joint astribot_arm_right_joint_4: limit lower=-0.052 upper=2.574 effort=45.0 velocity=5.0 -> lower=-0.053 upper=2.575 effort=45.0 velocity=5.0
- joint astribot_arm_right_joint_5: limit lower=-2.09 upper=2.108 effort=20.0 velocity=10.0 -> lower=-2.101 upper=2.101 effort=20.0 velocity=10.0
- joint astribot_arm_right_joint_6: limit lower=-0.76 upper=0.757 effort=8.0 velocity=5.0 -> lower=-0.75 upper=0.75 effort=8.0 velocity=5.0
- joint astribot_arm_right_joint_7: limit lower=-1.477 upper=1.447 effort=8.0 velocity=5.0 -> lower=-1.467 upper=1.467 effort=8.0 velocity=5.0

File: astribot_t1/model/urdf/astribot_torso.urdf (robot description, URDF)
Before this commit: robot astribot_torso, 6 links, 5 joints
Joints:
- joint astribot_torso_joint_4: limit lower=-1.627 upper=1.645 effort=200.0 velocity=3.0 -> lower=-1.636 upper=1.636 effort=200.0 velocity=3.0

File: astribot_t1/model/urdf/astribot_whole_body.urdf (robot description, URDF)
Before this commit: robot astribot_t1, 47 links, 46 joints
Joints:
- joint astribot_arm_left_joint_5: limit lower=-2.103 upper=2.098 effort=20.0 velocity=10.0 -> lower=-2.101 upper=2.101 effort=20.0 velocity=10.0
- joint astribot_arm_left_joint_6: limit lower=-0.755 upper=0.744 effort=8.0 velocity=5.0 -> lower=-0.75 upper=0.75 effort=8.0 velocity=5.0
- joint astribot_arm_left_joint_7: limit lower=-1.449 upper=1.485 effort=8.0 velocity=5.0 -> lower=-1.467 upper=1.467 effort=8.0 velocity=5.0
- joint astribot_arm_right_joint_1: limit lower=-1.606 upper=3.158 effort=80.0 velocity=3.0 -> lower=-1.579 upper=3.172 effort=80.0 velocity=3.0
- joint astribot_arm_right_joint_2: limit lower=-1.539 upper=0.192 effort=80.0 velocity=3.0 -> lower=-1.538 upper=0.201 effort=80.0 velocity=3.0
- joint astribot_arm_right_joint_3: limit lower=-0.741 upper=2.331 effort=40.0 velocity=3.0 -> lower=-0.745 upper=2.321 effort=40.0 velocity=3.0
- joint astribot_arm_right_joint_4: limit lower=-0.052 upper=2.574 effort=45.0 velocity=5.0 -> lower=-0.053 upper=2.575 effort=45.0 velocity=5.0
- joint astribot_arm_right_joint_5: limit lower=-2.09 upper=2.108 effort=20.0 velocity=10.0 -> lower=-2.101 upper=2.101 effort=20.0 velocity=10.0
- joint astribot_arm_right_joint_6: limit lower=-0.76 upper=0.757 effort=8.0 velocity=5.0 -> lower=-0.75 upper=0.75 effort=8.0 velocity=5.0
- joint astribot_arm_right_joint_7: limit lower=-1.477 upper=1.447 effort=8.0 velocity=5.0 -> lower=-1.467 upper=1.467 effort=8.0 velocity=5.0
- joint astribot_torso_joint_4: limit lower=-1.627 upper=1.645 effort=200.0 velocity=3.0 -> lower=-1.636 upper=1.636 effort=200.0 velocity=3.0

Commit message: release astribot_descriptions_github @ v0.0.0-dev

File: astribot_t1/model/urdf/astribot_arm_left.urdf (robot description, URDF)
Before this commit: robot astribot_arm_left, 9 links, 8 joints
Joints:
- joint astribot_arm_left_joint_1: limit lower=-3.172 upper=1.579 effort=80.0 velocity=3.0 -> lower=-3.172 upper=1.579 effort=80.0 velocity=3.5
- joint astribot_arm_left_joint_2: limit lower=-1.538 upper=0.201 effort=80.0 velocity=3.0 -> lower=-1.538 upper=0.201 effort=80.0 velocity=3.5
- joint astribot_arm_left_joint_3: limit lower=-2.321 upper=0.745 effort=40.0 velocity=3.0 -> lower=-2.321 upper=0.745 effort=40.0 velocity=3.5
- joint astribot_arm_left_joint_6: limit lower=-0.75 upper=0.75 effort=8.0 velocity=5.0 -> lower=-0.75 upper=0.75 effort=8.0 velocity=5.5
- joint astribot_arm_left_joint_7: limit lower=-1.467 upper=1.467 effort=8.0 velocity=5.0 -> lower=-1.467 upper=1.467 effort=8.0 velocity=5.5

File: astribot_t1/model/urdf/astribot_arm_right.urdf (robot description, URDF)
Before this commit: robot astribot_arm_right, 9 links, 8 joints
Joints:
- joint astribot_arm_right_joint_1: limit lower=-1.579 upper=3.172 effort=80.0 velocity=3.0 -> lower=-1.579 upper=3.172 effort=80.0 velocity=3.5
- joint astribot_arm_right_joint_2: limit lower=-1.538 upper=0.201 effort=80.0 velocity=3.0 -> lower=-1.538 upper=0.201 effort=80.0 velocity=3.5
- joint astribot_arm_right_joint_3: limit lower=-0.745 upper=2.321 effort=40.0 velocity=3.0 -> lower=-0.745 upper=2.321 effort=40.0 velocity=3.5
- joint astribot_arm_right_joint_6: limit lower=-0.75 upper=0.75 effort=8.0 velocity=5.0 -> lower=-0.75 upper=0.75 effort=8.0 velocity=5.5
- joint astribot_arm_right_joint_7: limit lower=-1.467 upper=1.467 effort=8.0 velocity=5.0 -> lower=-1.467 upper=1.467 effort=8.0 velocity=5.5

File: astribot_t1/model/urdf/astribot_whole_body.urdf (robot description, URDF)
Before this commit: robot astribot_t1, 47 links, 46 joints
Joints:
- joint astribot_arm_left_joint_1: limit lower=-3.172 upper=1.579 effort=80.0 velocity=3.0 -> lower=-3.172 upper=1.579 effort=80.0 velocity=3.5
- joint astribot_arm_left_joint_2: limit lower=-1.538 upper=0.201 effort=80.0 velocity=3.0 -> lower=-1.538 upper=0.201 effort=80.0 velocity=3.5
- joint astribot_arm_left_joint_3: limit lower=-2.321 upper=0.745 effort=40.0 velocity=3.0 -> lower=-2.321 upper=0.745 effort=40.0 velocity=3.5
- joint astribot_arm_left_joint_6: limit lower=-0.75 upper=0.75 effort=8.0 velocity=5.0 -> lower=-0.75 upper=0.75 effort=8.0 velocity=5.5
- joint astribot_arm_left_joint_7: limit lower=-1.467 upper=1.467 effort=8.0 velocity=5.0 -> lower=-1.467 upper=1.467 effort=8.0 velocity=5.5
- joint astribot_arm_right_joint_1: limit lower=-1.579 upper=3.172 effort=80.0 velocity=3.0 -> lower=-1.579 upper=3.172 effort=80.0 velocity=3.5
- joint astribot_arm_right_joint_2: limit lower=-1.538 upper=0.201 effort=80.0 velocity=3.0 -> lower=-1.538 upper=0.201 effort=80.0 velocity=3.5
- joint astribot_arm_right_joint_3: limit lower=-0.745 upper=2.321 effort=40.0 velocity=3.0 -> lower=-0.745 upper=2.321 effort=40.0 velocity=3.5
- joint astribot_arm_right_joint_6: limit lower=-0.75 upper=0.75 effort=8.0 velocity=5.0 -> lower=-0.75 upper=0.75 effort=8.0 velocity=5.5
- joint astribot_arm_right_joint_7: limit lower=-1.467 upper=1.467 effort=8.0 velocity=5.0 -> lower=-1.467 upper=1.467 effort=8.0 velocity=5.5
